File: RS14-BatLockPCB/RS14-BatLockPCB.brd (EAGLE design)
At the start: 38.7 x 43.2 mm, 19 parts, among them IC1 LM741D, Q1 2N3904

Commit message: Updated layouts for new hole sizes
Updated both boards to include proper sized holes for the screws (correction from 0.22" radius to 0.22" diamater clearance). This also includes some minor tweeks to clean up the board size a bit.
Parts:
- removed LLATCH, LRELAY: (no value), led:LED3MM
- added LLAT, LRLY: (no value), led:LED3MM
- moved R8 12.0 mm to (11.4, 38.1), turned to 270 degrees
- moved R7 5.71 mm to (28.6, 38.1), turned to 270 degrees
- moved BAT 2.54 mm to (16.5, 6.99)
- moved POW 2.54 mm to (23.5, 6.99)
Connections:
- removed net N$3: OFF.P2
- net GNDA: now also LLAT.K, OFF.P2; no longer LLATCH.K
- net N$7: now also LLAT.A; no longer LLATCH.A
- net N$8: now also LRLY.A; no longer LRELAY.A
- net RON: now also LRLY.K; no longer LRELAY.K
Routing:
- net RON: track 46.5 -> 58.0 mm, vias 3 -> 1
- net GNDA: track 22.5 -> 30.7 mm
- net N$8: track 11.1 -> 6.98 mm
- net VCC: track 19.7 -> 17.2 mm
- net V+: track 34.5 -> 31.9 mm
- net N$4: track 20.4 -> 19.0 mm
- net N$7: track 9.57 -> 8.25 mm, vias 1 -> 0
Other:
- board size 38.7 x 43.2 mm -> 38.7 x 40 mm
- board text added: "NOTE: ON sig. powers circuit in startup."
- board text added: "Renaud"
