File: RS14-LEDdriverPCB/LED_Slave_Board.sch (EAGLE design)
At the start: 26 parts, among them U1 PIC32MX250F128B-I/SP

Commit message: Revised Board and Schematic
Changed capacitor footprints and screw hole placement
Parts:
- C1, C4, C5, C7, C8: device rcl:C-US050-024X044 -> rcl:C-US050-045X075
Changed lines of the file:
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@@
 <part name="R1" library="rcl" deviceset="R-US_" device="0204/7" value="100"/>
 <part name="R2" library="rcl" deviceset="R-US_" device="0204/7" value="10K"/>
-<part name="C1" library="rcl" deviceset="C-US" device="050-024X044" value="22uF"/>
+<part name="C1" library="rcl" deviceset="C-US" device="050-045X075" value="22uF"/>
 <part name="C3" library="rcl" deviceset="C-US" device="025-040X050" value="0.1uF">
 <attribute name="DPN" value="445-8421-ND"/>
@@
 <part name="JP4" library="rs-molex-sherlock" deviceset="SHERLOCK-4P" device="VERTICAL"/>
 <part name="JP6" library="con-molex" deviceset="22-23-2021" device=""/>
-<part name="C4" library="rcl" deviceset="C-US" device="050-024X044" value="22uF"/>
+<part name="C4" library="rcl" deviceset="C-US" device="050-045X075" value="22uF"/>
 <part name="JP7" library="con-molex" deviceset="22-23-2021" device=""/>
-<part name="C5" library="rcl" deviceset="C-US" device="050-024X044" value="22uF"/>
-<part name="C7" library="rcl" deviceset="C-US" device="050-024X044" value="22uF"/>
-<part name="C8" library="rcl" deviceset="C-US" device="050-024X044" value="22uF"/>
+<part name="C5" library="rcl" deviceset="C-US" device="050-045X075" value="22uF"/>
+<part name="C7" library="rcl" deviceset="C-US" device="050-045X075" value="22uF"/>
+<part name="C8" library="rcl" deviceset="C-US" device="050-045X075" value="22uF"/>
 <part name="C2" library="rcl" deviceset="C-US" device="025-024X044" value="1uF"/>
 <part name="JP10" library="pinhead" deviceset="PINHD-1X2" device=""/>
